Commit message: modify camera angle

File: limo_ros2_pkgs/limo_description/urdf/limo_four_acker_ignition.xacro (robot description, xacro)
@@ -20,4 +20,11 @@
     <xacro:property name="wheel_length" value="0.001" />
     <xacro:property name="wheel_radius" value="0.045" />
+    <!-- CAMERA POSE PROPERTIES -->
+    <xacro:property name="cam_x" value="0.030" />
+    <xacro:property name="cam_y" value="0.0" />
+    <xacro:property name="cam_z" value="0.175" />
+    <xacro:property name="cam_roll" value="0.0" />
+    <xacro:property name="cam_pitch" value="0.5236" />
+    <xacro:property name="cam_yaw" value="0.0" />
   <link name="base_footprint"/>
   <joint name="base_joint" type="fixed">
@@ -59,5 +66,5 @@
     </xacro:limo_laser>
     <xacro:limo_depth_camera parent_prefix="base_link" frame_prefix="depth_camera">
-        <origin xyz="0.084 0 0.026" rpy="0 0 0"/>
+        <origin xyz="${cam_x} ${cam_y} ${cam_z}" rpy="${cam_roll} ${cam_pitch} ${cam_yaw}"/>
     </xacro:limo_depth_camera>
     <xacro:limo_imu parent_prefix="base_link" frame_prefix="imu">
@@ -268,4 +275,7 @@
       <child link="camera_depth_optical_frame" />
     </joint>
+    <gazebo reference="camera_depth_optical_joint">
+      <preserveFixedJoint>true</preserveFixedJoint>
+    </gazebo>
     <!-- gz-sim port; type="depth" -> type="rgbd_camera" (native color +
          depth + points + camera_info, no in-URDF plugin). -->
@@ -287,5 +297,5 @@
                 <far>10.0</far>
               </clip>
-              <optical_frame_id>depth_camera_link</optical_frame_id>
+              <optical_frame_id>camera_depth_optical_frame</optical_frame_id>
             </camera>
         </sensor>
